File: Tracer-S3.kicad_pcb (KiCad board)
At the start: 2 copper layers, 92.7 x 86.8 mm, 41 parts, among them J1 Conn_01x06_Socket, J2 Conn_02x02_Odd_Even, J3 Conn_02x02_Odd_Even, J4 Conn_02x02_Odd_Even, J5 Conn_02x02_Odd_Even, J6 Conn_02x04_Odd_Even, J7 Conn_01x02_Pin, Q1 BSP89, SW1 SW_Push, SW2 SW_Push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

Commit message: v2
Parts:
- added D4: D_Schottky, Diode_SMD:D_SOD-123, F.Cu at (128.3, 77.1)
- R10, R11, R2, R3, R4, R5, R6, R7, R8, R9: footprint Resistor_THT:R_Axial_DIN0204_L3.6mm_D1.6mm_P7.62mm_Horizontal -> Resistor_THT:R_Axial_DIN0207_L6.3mm_D2.5mm_P10.16mm_Horizontal
- moved J3 14.0 mm to (196.8, 80.0)
- moved J2 13.8 mm to (110.5, 80.2)
- moved S1 7.75 mm to (109.2, 119.5)
- moved S5 7.62 mm to (195.6, 119.4)
- moved R3 5.24 mm to (129.5, 48.3)
- moved R8 5.24 mm to (139.7, 48.3)
- moved R10 5.24 mm to (175.3, 48.3)
- moved R5 5.24 mm to (165.1, 48.3)
- moved S4 5.08 mm to (170.2, 53.3)
- moved D1 5.08 mm to (134.6, 44.7)
- moved D3 5.08 mm to (169.9, 44.7)
- moved S2 5.08 mm to (134.6, 53.3)
- moved R11 4.45 mm to (194.3, 93.3)
- moved R6 4.32 mm to (108.0, 93.5)
- moved J6 2.54 mm to (180.3, 96.5)
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Connections:
- Q1 pad 1: unconnected-(Q1-G-Pad1) -> /FET_GATE
- SW3 pad 1: +BATT -> Net-(D4-A)
- U1 pad 12: unconnected-(U1-GPIO8/TOUCH8/ADC1_CH7/SUBSPICS1-Pad12) -> /FET_GATE
Routing:
- net /FET_GATE: track 0.00 -> 69.8 mm, vias 0 -> 2
- net +3.3V: track 251.8 -> 309.9 mm
- net /FET_D: track 149.7 -> 202.5 mm
- net /S5: track 46.2 -> 67.8 mm
- net /S1: track 76.4 -> 97.9 mm
- net GND: track 7.60 -> 26.9 mm, vias 55 -> 53
- net Net-(S1-Anode): track 4.30 -> 13.9 mm
- net Net-(S5-Anode): track 4.30 -> 13.8 mm
- net Net-(D4-A): track 0.00 -> 5.61 mm
- net /LED1: track 59.2 -> 64.3 mm
- net /S2: track 70.2 -> 73.1 mm
- net /S3: track 58.5 -> 56.3 mm
- net /MODE: track 9.23 -> 8.17 mm
- net /BIN2: track 8.20 -> 9.25 mm
- net /BIN1: track 7.67 -> 8.72 mm
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Other:
- board size 92.7 x 86.8 mm -> 92.5 x 86.9 mm
- board text added: "MOS@53175DDD Tracer-S3 v2"
- board text removed: "MOS@53175DDD Tracer-S3 v1"

Commit message: 部品番号修正
Parts:
- R10, R11, R8, R9: value R -> 33k
- R2, R3, R4, R5: value R -> 47R
- R6: renamed from R7; value R -> 47R
- R7: renamed from R6; value R -> 33k
Changed lines of the file:
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@@
         (effects (font (size 1 1) (thickness 0.15)))
     )
-    (fp_text value "R" (at 5.08 2.37 -90) (layer "F.Fab")
+    (fp_text value "47R" (at 5.08 2.37 -90) (layer "F.Fab")
         (effects (font (size 1 1) (thickness 0.15)))
     )
@@
     (property "ki_keywords" "R res resistor")
     (attr through_hole)
-    (fp_text reference "R6" (at 5.08 0 -90) (layer "F.SilkS")
-        (effects (font (size 1 1) (thickness 0.15)))
-    )
-    (fp_text value "R" (at 5.08 2.37 -90) (layer "F.Fab")
+    (fp_text reference "R7" (at 5.08 0 -90) (layer "F.SilkS")
+        (effects (font (size 1 1) (thickness 0.15)))
+    )
+    (fp_text value "33k" (at 5.08 2.37 -90) (layer "F.Fab")
         (effects (font (size 1 1) (thickness 0.15)))
     )
@@
     (descr "Resistor SMD 0603 (1608 Metric), square (rectangular) end terminal, IPC_7351 nominal, (Body size source: IPC-SM-782 page 72, https://www.pcb-3d.com/wordpress/wp-content/uploads/ipc-sm-782a_amendment_1_and_2.pdf), generated with kicad-footprint-generator")
     (tags "resistor")
-    (property "LCSC" "C3017715")
+    (property "LCSC" "C269701")
     (property "Sheetfile" "Tracer-S3.kicad_sch")
     (property "Sheetname" "")
@@
         (effects (font (size 1 1) (thickness 0.15)))
     )
-    (fp_text value "R" (at 5.08 2.37 -90) (layer "F.Fab")
+    (fp_text value "33k" (at 5.08 2.37 -90) (layer "F.Fab")
         (effects (font (size 1 1) (thickness 0.15)))
     )
@@
         (effects (font (size 1 1) (thickness 0.15)))
     )
-    (fp_text value "R" (at 5.08 2.37 -90) (layer "F.Fab")
+    (fp_text value "33k" (at 5.08 2.37 -90) (layer "F.Fab")
         (effects (font (size 1 1) (thickness 0.15)))
     )
@@
     (descr "Resistor SMD 0603 (1608 Metric), square (rectangular) end terminal, IPC_7351 nominal, (Body size source: IPC-SM-782 page 72, https://www.pcb-3d.com/wordpress/wp-content/uploads/ipc-sm-782a_amendment_1_and_2.pdf), generated with kicad-footprint-generator")
     (tags "resistor")
-    (property "LCSC" "C3017715")
+    (property "LCSC" "C269701")
     (property "Sheetfile" "Tracer-S3.kicad_sch")
     (property "Sheetname" "")
@@
         (effects (font (size 1 1) (thickness 0.15)))
     )
-    (fp_text value "R" (at 5.08 2.37 -90) (layer "F.Fab")
+    (fp_text value "47R" (at 5.08 2.37 -90) (layer "F.Fab")
         (effects (font (size 1 1) (thickness 0.15)))
     )
@@
     (property "ki_keywords" "R res resistor")
     (attr through_hole)
-    (fp_text reference "R7" (at 5.08 0 270 unlocked) (layer "F.SilkS")
-        (effects (font (size 1 1) (thickness 0.15)))
-    )
-    (fp_text value "R" (at 5.08 2.37 90) (layer "F.Fab")
+    (fp_text reference "R6" (at 5.08 0 270 unlocked) (layer "F.SilkS")
+        (effects (font (size 1 1) (thickness 0.15)))
+    )
+    (fp_text value "47R" (at 5.08 2.37 90) (layer "F.Fab")
         (effects (font (size 1 1) (thickness 0.15)))
     )
@@
     (descr "Resistor SMD 0603 (1608 Metric), square (rectangular) end terminal, IPC_7351 nominal, (Body size source: IPC-SM-782 page 72, https://www.pcb-3d.com/wordpress/wp-content/uploads/ipc-sm-782a_amendment_1_and_2.pdf), generated with kicad-footprint-generator")
     (tags "resistor")
-    (property "LCSC" "C3017715")
+    (property "LCSC" "C269701")
     (property "Sheetfile" "Tracer-S3.kicad_sch")
     (property "Sheetname" "")
@@
     (descr "Resistor SMD 0603 (1608 Metric), square (rectangular) end terminal, IPC_7351 nominal, (Body size source: IPC-SM-782 page 72, https://www.pcb-3d.com/wordpress/wp-content/uploads/ipc-sm-782a_amendment_1_and_2.pdf), generated with kicad-footprint-generator")
     (tags "resistor")
-    (property "LCSC" "C3017715")
+    (property "LCSC" "C269701")
     (property "Sheetfile" "Tracer-S3.kicad_sch")
     (property "Sheetname" "")
@@
         (effects (font (size 1 1) (thickness 0.15)))
     )
-    (fp_text value "R" (at 5.08 2.37 -90) (layer "F.Fab")
+    (fp_text value "33k" (at 5.08 2.37 -90) (layer "F.Fab")
         (effects (font (size 1 1) (thickness 0.15)))
     )
@@
         (effects (font (size 1 1) (thickness 0.15)))
     )
-    (fp_text value "R" (at 5.08 2.37 -90) (layer "F.Fab")
+    (fp_text value "33k" (at 5.08 2.37 -90) (layer "F.Fab")
         (effects (font (size 1 1) (thickness 0.15)))
     )
@@
         (effects (font (size 1 1) (thickness 0.15)))
     )
-    (fp_text value "R" (at 5.08 2.37 -90) (layer "F.Fab")
+    (fp_text value "47R" (at 5.08 2.37 -90) (layer "F.Fab")
         (effects (font (size 1 1) (thickness 0.15)))
     )
@@
     (descr "Resistor SMD 0603 (1608 Metric), square (rectangular) end terminal, IPC_7351 nominal, (Body size source: IPC-SM-782 page 72, https://www.pcb-3d.com/wordpress/wp-content/uploads/ipc-sm-782a_amendment_1_and_2.pdf), generated with kicad-footprint-generator")
     (tags "resistor")
-    (property "LCSC" "C3017715")
+    (property "LCSC" "C269701")
     (property "Sheetfile" "Tracer-S3.kicad_sch")
     (property "Sheetname" "")
@@
         (effects (font (size 1 1) (thickness 0.15)))
     )
-    (fp_text value "R" (at 5.08 2.37 90) (layer "F.Fab")
-        (effects (font (size 1 1) (thickness 0.15)))
-    )
+    (fp_text value "47R" (at 5.08 2.37 90) (layer "F.Fab")
+        (effects (font (size 1 1) (thickness 0.15)))
+    )

Commit message: 回路定数変更
Parts:
- R10, R11, R7, R8, R9: value 33k -> 10k
Changed lines of the file:
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@@
         (effects (font (size 1 1) (thickness 0.15)))
     )
-    (fp_text value "33k" (at 5.08 2.37 -90) (layer "F.Fab")
+    (fp_text value "10k" (at 5.08 2.37 -90) (layer "F.Fab")
         (effects (font (size 1 1) (thickness 0.15)))
     )
@@
         (effects (font (size 1 1) (thickness 0.15)))
     )
-    (fp_text value "33k" (at 5.08 2.37 -90) (layer "F.Fab")
+    (fp_text value "10k" (at 5.08 2.37 -90) (layer "F.Fab")
         (effects (font (size 1 1) (thickness 0.15)))
     )
@@
         (effects (font (size 1 1) (thickness 0.15)))
     )
-    (fp_text value "33k" (at 5.08 2.37 -90) (layer "F.Fab")
+    (fp_text value "10k" (at 5.08 2.37 -90) (layer "F.Fab")
         (effects (font (size 1 1) (thickness 0.15)))
     )
@@
         (effects (font (size 1 1) (thickness 0.15)))
     )
-    (fp_text value "33k" (at 5.08 2.37 -90) (layer "F.Fab")
+    (fp_text value "10k" (at 5.08 2.37 -90) (layer "F.Fab")
         (effects (font (size 1 1) (thickness 0.15)))
     )
@@
         (effects (font (size 1 1) (thickness 0.15)))
     )
-    (fp_text value "33k" (at 5.08 2.37 -90) (layer "F.Fab")
-        (effects (font (size 1 1) (thickness 0.15)))
-    )
+    (fp_text value "10k" (at 5.08 2.37 -90) (layer "F.Fab")
+        (effects (font (size 1 1) (thickness 0.15)))
+    )

Commit message: センサ間隔調整・外形修正
Parts:
- moved D1 1.91 mm to (132.7, 44.7)
- moved D3 1.91 mm to (171.8, 44.7)
- moved R10 1.91 mm to (177.2, 48.3)
- moved R5 1.91 mm to (167.0, 48.3)
- moved R8 1.91 mm to (137.8, 48.3)
- moved S2 1.91 mm to (132.7, 53.3)
- moved S4 1.91 mm to (172.1, 53.3)
- moved R3 1.90 mm to (127.6, 48.3)
Routing:
- net +3.3V: track 309.9 -> 290.3 mm
- net /S4: track 57.7 -> 48.4 mm
- net /FET_D: track 202.5 -> 206.3 mm
- net /LED1: track 64.3 -> 66.2 mm
- net /S2: track 73.1 -> 75.0 mm
- net /LED3: track 45.4 -> 46.2 mm
Other:
- outline, holes or cut-outs redrawn

Commit message: 電源スイッチ配線変更・ミシン穴追加
Connections:
- SW3 pad 3: unconnected-(SW3-C-Pad3) -> Net-(J7-Pin_1)
Routing:
- net Net-(J7-Pin_1): track 8.43 -> 7.66 mm
Other:
- outline, holes or cut-outs redrawn
